Commit message: [update]修改了launch文件，增强其可读性

File: src/rm_nav_bringup/urdf/sentry_robot_sim.xacro (robot description, xacro)
@@ -136,5 +136,5 @@
   <joint name="imu_joint" type="fixed">
     <axis xyz="0 1 0" />
-    <origin xyz="0.12 0 0.125" rpy="0 0 0"/>
+    <origin xyz="$(arg xyz)" rpy="$(arg rpy)"/>
     <parent link="base_link"/>
     <child link="imu_link"/>

Commit message: feat(nav): harden small-gicp startup and add configurable lidar noise

File: src/rm_nav_bringup/urdf/sentry_robot_sim.xacro (robot description, xacro)
@@ -17,4 +17,5 @@
   <xacro:arg name="right_xyz" default="0.12 -0.14 0.175" />
   <xacro:arg name="right_rpy" default="0 0 -0.610865" />
+  <xacro:arg name="lidar_noise_stddev" default="0.002" />
   <link name="dummy"/>
   <link name="base_link">
@@ -237,9 +238,11 @@
   <!-- Livox-Mid360  -->
   <xacro:include filename="$(find ros2_livox_simulation)/urdf/mid360.xacro" />
-  <xacro:mid360 name="livox_frame" parent="base_link" topic="/livox/lidar">
+  <xacro:mid360 name="livox_frame" parent="base_link" topic="/livox/lidar"
+    noise_stddev="$(arg lidar_noise_stddev)">
     <origin xyz="$(arg xyz)" rpy="$(arg rpy)" />
   </xacro:mid360>
   <xacro:if value="$(arg dual_lidar)">
-    <xacro:mid360 name="livox_right_frame" parent="base_link" topic="/livox_right/lidar">
+    <xacro:mid360 name="livox_right_frame" parent="base_link" topic="/livox_right/lidar"
+      noise_stddev="$(arg lidar_noise_stddev)">
       <origin xyz="$(arg right_xyz)" rpy="$(arg right_rpy)" />
     </xacro:mid360>

File: src/rm_simulation/livox_laser_simulation_RO2/urdf/mid360.xacro (robot description, xacro)
@@ -19,5 +19,5 @@
     </inertial>
   </xacro:macro>
-  <xacro:macro name="mid360" params="name:='' parent:= 'base_link' topic:='mid360' *origin ">
+  <xacro:macro name="mid360" params="name:='' parent:= 'base_link' topic:='mid360' noise_mean:='0.0' noise_stddev:='0.002' *origin ">
     <link name="${name}">
       <visual>
