Commit message: nav2: add dual-lidar consume switch and stabilize RMUL26 dual run

File: src/rm_nav_bringup/urdf/sentry_robot_real.xacro (robot description, xacro)
@@ -11,7 +11,10 @@
     </inertial>
   </xacro:macro>
-  <!-- base_link to livox_frame -->
+  <!-- base_link to primary livox_frame -->
   <xacro:arg name="xyz" default="0.0 0.045 0.49" />
   <xacro:arg name="rpy" default="0 0 0" />
+  <xacro:arg name="dual_lidar" default="false" />
+  <xacro:arg name="right_xyz" default="0.12 -0.14 0.49" />
+  <xacro:arg name="right_rpy" default="0 0 -0.610865" />
   <link name="base_link">
     <visual>
@@ -145,3 +148,21 @@
     <child link="livox_frame"/>
   </joint>
+  <xacro:if value="$(arg dual_lidar)">
+    <link name="livox_right_frame">
+      <visual>
+        <origin xyz="0.025 -0.0265 -0.025" rpy="${pi/2} 0 ${pi}"/>
+        <geometry>
+          <mesh filename="package://pb_rm_simulation/meshes/mid360.stl" scale="0.001 0.001 0.001"/>
+        </geometry>
+        <material name="blue">
+          <color rgba="0 0 1.0 1" />
+        </material>
+      </visual>
+    </link>
+    <joint name="livox_right_joint" type="fixed">
+      <origin xyz="$(arg right_xyz)" rpy="$(arg right_rpy)" />
+      <parent link="base_link"/>
+      <child link="livox_right_frame"/>
+    </joint>
+  </xacro:if>
 </robot>

File: src/rm_nav_bringup/urdf/sentry_robot_sim.xacro (robot description, xacro)
@@ -11,7 +11,10 @@
     </inertial>
   </xacro:macro>
-  <!-- base_link to livox_frame -->
+  <!-- base_link to primary livox_frame -->
   <xacro:arg name="xyz" default="0.12 0.0 0.175" />
   <xacro:arg name="rpy" default="0 0 0" />
+  <xacro:arg name="dual_lidar" default="false" />
+  <xacro:arg name="right_xyz" default="0.12 -0.14 0.175" />
+  <xacro:arg name="right_rpy" default="0 0 -0.610865" />
   <link name="dummy"/>
   <link name="base_link">
@@ -185,4 +188,9 @@
     <material>Gazebo/LightBlueLaser</material>
   </gazebo>
+  <xacro:if value="$(arg dual_lidar)">
+    <gazebo reference="livox_right_frame">
+      <material>Gazebo/LightBlueLaser</material>
+    </gazebo>
+  </xacro:if>
   <!-- Drive controller plugin-->
   <!-- https://github.com/ros-simulation/gazebo_ros_pkgs/wiki/ROS-2-Migration:-Planar-Move -->
@@ -232,3 +240,8 @@
     <origin xyz="$(arg xyz)" rpy="$(arg rpy)" />
   </xacro:mid360>
+  <xacro:if value="$(arg dual_lidar)">
+    <xacro:mid360 name="livox_right_frame" parent="base_link" topic="/livox_right/lidar">
+      <origin xyz="$(arg right_xyz)" rpy="$(arg right_rpy)" />
+    </xacro:mid360>
+  </xacro:if>
 </robot>

Commit message: fix(bringup): warn mapping+nav2 mixed mode and avoid broken lidar mesh

File: src/rm_nav_bringup/urdf/sentry_robot_real.xacro (robot description, xacro)
@@ -134,7 +134,8 @@
   <link name="livox_frame">
     <visual>
-      <origin xyz="0.025 -0.0265 -0.025" rpy="${pi/2} 0 ${pi}"/>
+      <origin xyz="0.0 0.0 0.0" rpy="0 0 0"/>
       <geometry>
-        <mesh filename="package://pb_rm_simulation/meshes/mid360.stl" scale="0.001 0.001 0.001"/>
+        <!-- Use primitive geometry to avoid RViz stalls when external STL assets are unavailable/corrupted. -->
+        <cylinder length="0.06" radius="0.035"/>
       </geometry>
       <material name="blue">
@@ -151,7 +152,8 @@
     <link name="livox_right_frame">
       <visual>
-        <origin xyz="0.025 -0.0265 -0.025" rpy="${pi/2} 0 ${pi}"/>
+        <origin xyz="0.0 0.0 0.0" rpy="0 0 0"/>
         <geometry>
-          <mesh filename="package://pb_rm_simulation/meshes/mid360.stl" scale="0.001 0.001 0.001"/>
+          <!-- Keep same placeholder for right lidar visual. -->
+          <cylinder length="0.06" radius="0.035"/>
         </geometry>
         <material name="blue">
